File: Hardware/5V_WS2812_N_SERVO.kicad_sch (KiCad schematic)
At the start: 6 parts, among them J4 Servo1, J5 Screw_Terminal_01x03, U8 SN74LVC1G00DBV

Commit message: Finish PCB
Changed lines of the file:
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@@
 		)
 	)
-	(hierarchical_label "Other{5VPWM BUZZER LED}"
+	(hierarchical_label "Other{5VPWM USER_SW LED}"
 		(shape input)
 		(at 71.12 86.36 180)
