File: Hardware/Bells and whistles.kicad_sch (KiCad schematic)
At the start: 2 parts

Commit message: Finish PCB
Changed lines of the file:
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@@
-		)
-	)
-	(bus_entry
-		(at 119.38 74.93)
-		(size 2.54 2.54)
-		(stroke
-			(width 0)
-			(type default)
 		)
 	)
 	(bus
 		(pts
-			(xy 119.38 73.66) (xy 119.38 74.93)
+			(xy 119.38 73.66) (xy 119.38 77.47)
 		)
 		(stroke
@@
 		(pts
 			(xy 110.49 73.66) (xy 119.38 73.66)
-		)
-		(stroke
-			(width 0)
-			(type default)
-		)
-	)
-	(bus
-		(pts
-			(xy 119.38 74.93) (xy 119.38 77.47)
-		)
-		(stroke
-			(width 0)
-			(type default)
-		)
-	)
-	(wire
-		(pts
-			(xy 121.92 77.47) (xy 137.16 77.47)
 		)
 		(stroke
@@
 		)
 	)
-	(label "Other.BUZZER"
-		(at 137.16 77.47 0)
-		(fields_autoplaced yes)
-		(effects
-			(font
-				(size 1.27 1.27)
-			)
-			(justify left bottom)
-		)
-	)
 	(label "Other.LED"
 		(at 181.61 83.82 0)
@@
 		)
 	)
-	(hierarchical_label "Other{5VPWM BUZZER LED}"
+	(hierarchical_label "Other{5VPWM USER_SW LED}"
 		(shape input)
 		(at 110.49 73.66 180)
