File: Hardware/ESP32S3.kicad_sch (KiCad schematic)
At the start: 4 parts, among them U22 ESP32-S3-WROOM-1

Commit message: Finish PCB
Changed lines of the file:
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@@
-		)
-	)
-	(label "Other.BUZZER"
-		(at 58.42 73.66 0)
-		(fields_autoplaced yes)
-		(effects
-			(font
-				(size 1.27 1.27)
-			)
-			(justify left bottom)
 		)
 	)
@@
 		)
 	)
-	(label "Other.BUZZER"
+	(label "Other.USER_SW"
 		(at 219.71 144.78 0)
 		(fields_autoplaced yes)
@@
 	(label "IO47"
 		(at 151.13 124.46 0)
+		(fields_autoplaced yes)
+		(effects
+			(font
+				(size 1.27 1.27)
+			)
+			(justify left bottom)
+		)
+	)
+	(label "Other.USER_SW"
+		(at 58.42 73.66 0)
 		(fields_autoplaced yes)
 		(effects
@@
 		)
 	)
-	(hierarchical_label "Other{5VPWM BUZZER LED}"
+	(hierarchical_label "Other{5VPWM USER_SW LED}"
 		(shape input)
 		(at 242.57 139.7 0)
