File: Hardware/MCU.kicad_sch (KiCad schematic)
At the start: 0 parts

Commit message: Finish PCB
Other:
- sheet 5V WS2812 and Servo ports: added Other{5VPWM USER_SW LED}; removed Other{5VPWM BUZZER LED}
- sheet Bells and whistles ports: added Other{5VPWM USER_SW LED}; removed Other{5VPWM BUZZER LED}
- sheet ESP32S3 ports: added Other{5VPWM USER_SW LED}; removed Other{5VPWM BUZZER LED}
- sheet POWER SECTION ports: added Other{5VPWM USER_SW LED}; removed none
Changed lines of the file:
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@@
 	(bus
 		(pts
-			(xy 176.53 66.04) (xy 200.66 66.04)
+			(xy 176.53 63.5) (xy 200.66 63.5)
+		)
+		(stroke
+			(width 0)
+			(type default)
+		)
+	)
+	(bus
+		(pts
+			(xy 200.66 68.58) (xy 186.69 68.58)
 		)
 		(stroke
@@
 		(pts
 			(xy 57.15 46.99) (xy 64.77 46.99)
+		)
+		(stroke
+			(width 0)
+			(type default)
+		)
+	)
+	(bus
+		(pts
+			(xy 186.69 68.58) (xy 186.69 87.63)
 		)
 		(stroke
@@
 			)
 		)
-		(pin "Other{5VPWM BUZZER LED}" input
+		(pin "Other{5VPWM USER_SW LED}" input
 			(at 200.66 87.63 180)
 			(effects
@@
 			)
 		)
-		(pin "Other{5VPWM BUZZER LED}" input
-			(at 176.53 87.63 0)
-			(effects
-				(font
-					(size 1.27 1.27)
-				)
-				(justify right)
-			)
-		)
 		(pin "Hbridge3{IN1 IN2}" input
 			(at 176.53 57.15 0)
@@
 		)
 		(pin "I2C1{SCL SDA}" input
-			(at 176.53 66.04 0)
+			(at 176.53 63.5 0)
 			(effects
 				(font
@@
 				)
 				(justify left)
+			)
+		)
+		(pin "Other{5VPWM USER_SW LED}" input
+			(at 176.53 87.63 0)
+			(effects
+				(font
+					(size 1.27 1.27)
+				)
+				(justify right)
 			)
 		)
@@
 			)
 		)
-		(pin "Other{5VPWM BUZZER LED}" input
+		(pin "Other{5VPWM USER_SW LED}" input
 			(at 200.66 113.03 180)
 			(effects
@@
 		)
 		(pin "I2C1{SCL SDA}" input
-			(at 200.66 66.04 180)
-			(effects
-				(font
+			(at 200.66 63.5 180)
+			(effects
+				(font
+					(size 1.27 1.27)
+				)
+				(justify left)
+			)
+		)
+		(pin "Other{5VPWM USER_SW LED}" input
+			(at 200.66 68.58 180)
+			(effects
+				(font
