File: Hardware/POWER.kicad_sch (KiCad schematic)
At the start: 4 parts

Commit message: Finish PCB
Parts:
- added R12: 10kΩ, PCM_JLCPCB:R_0402, symbol PCM_JLCPCB-Resistors:0402,10kΩ
Connections:
- net DRV1/~{SAFE OPERATION}: no longer S1.1
- net GND: now also R12.2
- new net Other.USER_SW: R12.1, S1.1
