File: PCB source/SimpleLedController.kicad_pcb (KiCad board)
At the start: 4 copper layers, 90 x 50 mm, 181 parts, among them J1 Jack-DC, J12 Screw_Terminal_01x02, J13 Screw_Terminal_01x02, J14 Screw_Terminal_01x02, J2 Molex KK2.54 4p male, J3 Connector, USB-TYPE-C-16P, J4 Servo1, J5 Screw_Terminal_01x03, J6 Conn_01x06, Q10 AO3400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

Commit message: Remove boardhouse designators
Parts:
- added REF**: My_github, Symbol:My_github, B.Cu at (139.2, 94.5)
Other:
- board text removed: "JLCJLCJLCJLC"
- board text removed: "MADE IN CHINA BY JLCPCB"
